Commit message: added controller manager and its config

File: description/gazebo_control.xacro (robot description, xacro)
@@ -1,21 +1,23 @@
 <?xml version="1.0"?>
 <robot xmlns:xacro="http://www.ros.org/wiki/xacro">
-    <gazebo>
-        <plugin name='diff_drive' filename='libgazebo_ros_diff_drive.so'>
-            <!-- Wheel Information -->
-            <left_joint>left_wheel_joint</left_joint>
-            <right_joint>right_wheel_joint</right_joint>
-            <wheel_separation>0.35</wheel_separation>
-            <wheel_diameter>0.1</wheel_diameter>
-            <!-- Limits -->
-            <max_wheel_torque>200</max_wheel_torque>
-            <max_wheel_acceleration>10.0</max_wheel_acceleration>
-            <!-- Output -->
-            <odometry_frame>odom</odometry_frame>
-            <robot_base_frame>base_link</robot_base_frame>
-            <publish_odom>true</publish_odom>
-            <publish_odom_tf>true</publish_odom_tf>
-            <publish_wheel_tf>true</publish_wheel_tf>
-        </plugin>
-    </gazebo>
+    <xacro:macro name="gazebo_control" params="">
+        <gazebo>
+            <plugin name='diff_drive' filename='libgazebo_ros_diff_drive.so'>
+                <!-- Wheel Information -->
+                <left_joint>left_wheel_joint</left_joint>
+                <right_joint>right_wheel_joint</right_joint>
+                <wheel_separation>0.35</wheel_separation>
+                <wheel_diameter>0.1</wheel_diameter>
+                <!-- Limits -->
+                <max_wheel_torque>200</max_wheel_torque>
+                <max_wheel_acceleration>10.0</max_wheel_acceleration>
+                <!-- Output -->
+                <odometry_frame>odom</odometry_frame>
+                <robot_base_frame>base_link</robot_base_frame>
+                <publish_odom>true</publish_odom>
+                <publish_odom_tf>true</publish_odom_tf>
+                <publish_wheel_tf>true</publish_wheel_tf>
+            </plugin>
+        </gazebo>
+    </xacro:macro>
 </robot>

File: description/imu.xacro (robot description, xacro)
@@ -1,58 +1,60 @@
 <?xml version="1.0"?>
 <robot xmlns:xacro="http://www.ros.org/wiki/xacro">
-  <!-- Joint connecting IMU to the robot -->
-  <joint name="imu_joint" type="fixed">
-    <parent link="chassis"/>
-    <child link="imu_frame"/>
-    <origin xyz="0.305 0 0.08" rpy="0 0 0"/>
-  </joint>
-  <!-- IMU link -->
-  <link name="imu_frame">
-    <visual>
-      <geometry>
-        <box size="0.010 0.03 0.03"/>
-      </geometry>
-      <material name="red"/>
-    </visual>
-    <collision>
-      <geometry>
-        <box size="0.03899 0.03785 0.01338"/>
-      </geometry>
-    </collision>
-    <inertial>
-      <origin xyz="0 0 0" rpy="0 0 0"/>
-      <mass value="0.031"/>
-      <inertia
-        ixx="6.22969e-06"
-        ixy="0.0"
-        ixz="0.0"
-        iyy="5.92858e-06"
-        iyz="0.0"
-        izz="9.15545e-06"/>
-    </inertial>
-  </link>
-  <!-- Material definition -->
-  <material name="imu_black">
-    <color rgba="0.1 0.1 0.1 1"/>
-  </material>
-  <!-- Gazebo sensor plugin -->
-  <gazebo reference="imu_frame">
-    <material>Gazebo/Red</material>
-    <sensor name="imu_sensor" type="imu">
-      <pose>0 0 0 0 0 0</pose>
-      <update_rate>15.0</update_rate>
-      <visualize>false</visualize>
-      <always_on>true</always_on>
-      <topic>imu/data</topic>
-      <gz_frame_id>imu_frame</gz_frame_id>
-      <!-- Plugin block -->
-      <plugin name="imu_controller" filename="libgazebo_ros_imu_sensor.so">
-        <ros>
-          <namespace>/</namespace>
-          <remapping>~/out:=imu</remapping>
-        </ros>
-        <frame_name>imu_frame</frame_name>
-      </plugin>
-    </sensor>
-  </gazebo>
+  <xacro:macro name="imu" params="">
+    <!-- Joint connecting IMU to the robot -->
+    <joint name="imu_joint" type="fixed">
+      <parent link="chassis"/>
+      <child link="imu_frame"/>
+      <origin xyz="0.305 0 0.08" rpy="0 0 0"/>
+    </joint>
+    <!-- IMU link -->
+    <link name="imu_frame">
+      <visual>
+        <geometry>
+          <box size="0.010 0.03 0.03"/>
+        </geometry>
+        <material name="red"/>
+      </visual>
+      <collision>
+        <geometry>
+          <box size="0.03899 0.03785 0.01338"/>
+        </geometry>
+      </collision>
+      <inertial>
+        <origin xyz="0 0 0" rpy="0 0 0"/>
+        <mass value="0.031"/>
+        <inertia
+          ixx="6.22969e-06"
+          ixy="0.0"
+          ixz="0.0"
+          iyy="5.92858e-06"
+          iyz="0.0"
+          izz="9.15545e-06"/>
+      </inertial>
+    </link>
+    <!-- Material definition -->
+    <material name="imu_black">
+      <color rgba="0.1 0.1 0.1 1"/>
+    </material>
+    <!-- Gazebo sensor plugin -->
+    <gazebo reference="imu_frame">
+      <material>Gazebo/Red</material>
+      <sensor name="imu_sensor" type="imu">
+        <pose>0 0 0 0 0 0</pose>
+        <update_rate>15.0</update_rate>
+        <visualize>false</visualize>
+        <always_on>true</always_on>
+        <topic>imu/data</topic>
+        <gz_frame_id>imu_frame</gz_frame_id>
+        <!-- Plugin block -->
+        <plugin name="imu_controller" filename="libgazebo_ros_imu_sensor.so">
+          <ros>
+            <namespace>/</namespace>
+            <remapping>~/out:=imu</remapping>
+          </ros>
+          <frame_name>imu_frame</frame_name>
+        </plugin>
+      </sensor>
+    </gazebo>
+  </xacro:macro>
 </robot>

File: description/lidar.xacro (robot description, xacro)
@@ -1,52 +1,54 @@
 <?xml version="1.0"?>
 <robot xmlns:xacro="http://www.ros.org/wiki/xacro" >
-    <joint name="laser_joint" type="fixed">
-        <parent link="chassis"/>
-        <child link="laser_frame"/>
-        <origin xyz="0.1 0 0.175" rpy="0 0 0"/>
-    </joint>
-    <link name="laser_frame">
-        <visual>
-            <geometry>
-                <cylinder radius="0.05" length="0.04"/>
-            </geometry>
-            <material name="red"/>
-        </visual>
-        <collision>
-            <geometry>
-                <cylinder radius="0.05" length="0.04"/>
-            </geometry>
-        </collision>
-        <xacro:inertial_cylinder mass="0.1" length="0.04" radius="0.05">
-            <origin xyz="0 0 0" rpy="0 0 0"/>
-        </xacro:inertial_cylinder>
-    </link>
-    <gazebo reference="laser_frame">
-        <material>Gazebo/Red</material>
-        <sensor name="laser" type="ray">
-            <pose> 0 0 0 0 0 0 </pose>
-            <visualize>true</visualize>
-            <update_rate>10</update_rate>
-            <ray>
-                <scan>
-                    <horizontal>
-                        <samples>360</samples>
-                        <min_angle>-3.14</min_angle>
-                        <max_angle>3.14</max_angle>
-                    </horizontal>
-                </scan>
-                <range>
-                    <min>0.3</min>
-                    <max>12</max>
-                </range>
-            </ray>
-            <plugin name="laser_controller" filename="libgazebo_ros_ray_sensor.so">
-                <ros>
-                    <argument>~/out:=scan</argument>
-                </ros>
-                <output_type>sensor_msgs/LaserScan</output_type>
-                <frame_name>laser_frame</frame_name>
-            </plugin>
-        </sensor>
-    </gazebo>
+    <xacro:macro name="lidar" params="">
+        <joint name="laser_joint" type="fixed">
+            <parent link="chassis"/>
+            <child link="laser_frame"/>
+            <origin xyz="0.1 0 0.175" rpy="0 0 0"/>
+        </joint>
+        <link name="laser_frame">
+            <visual>
+                <geometry>
+                    <cylinder radius="0.05" length="0.04"/>
+                </geometry>
+                <material name="red"/>
+            </visual>
+            <collision>
+                <geometry>
+                    <cylinder radius="0.05" length="0.04"/>
+                </geometry>
+            </collision>
+            <xacro:inertial_cylinder mass="0.1" length="0.04" radius="0.05">
+                <origin xyz="0 0 0" rpy="0 0 0"/>
+            </xacro:inertial_cylinder>
+        </link>
+        <gazebo reference="laser_frame">
+            <material>Gazebo/Red</material>
+            <sensor name="laser" type="ray">
+                <pose> 0 0 0 0 0 0 </pose>
+                <visualize>true</visualize>
+                <update_rate>10</update_rate>
+                <ray>
+                    <scan>
+                        <horizontal>
+                            <samples>360</samples>
+                            <min_angle>-3.14</min_angle>
+                            <max_angle>3.14</max_angle>
+                        </horizontal>
+                    </scan>
+                    <range>
+                        <min>0.3</min>
+                        <max>12</max>
+                    </range>
+                </ray>
+                <plugin name="laser_controller" filename="libgazebo_ros_ray_sensor.so">
+                    <ros>
+                        <argument>~/out:=scan</argument>
+                    </ros>
+                    <output_type>sensor_msgs/LaserScan</output_type>
+                    <frame_name>laser_frame</frame_name>
+                </plugin>
+            </sensor>
+        </gazebo>
+    </xacro:macro>
 </robot>

File: description/robot.urdf.xacro (robot description, xacro)
@@ -2,6 +2,11 @@
 <robot xmlns:xacro="http://www.ros.org/wiki/xacro"  name="robot">
     <xacro:include filename="robot_core.xacro" />
-    <xacro:include filename="gazebo_control.xacro" />
+    <!--<xacro:include filename="gazebo_control.xacro" /> -->
     <xacro:include filename="lidar.xacro" />
     <xacro:include filename="imu.xacro" />
+    <xacro:robot_core/>
+    <xacro:lidar/>
+    <xacro:imu/>
+    <!-- <xacro:gazebo_control/> -->
+    <xacro:include filename="ros2_control.xacro" />
 </robot>

File: description/robot_core.xacro (robot description, xacro)
@@ -2,118 +2,120 @@
 <robot xmlns:xacro="http://www.ros.org/wiki/xacro" >
     <xacro:include filename="inertial_macros.xacro"/>
-    <material name="white">
-        <color rgba="1 1 1 1" />
-    </material>
-    <material name="orange">
-        <color rgba="1 0.3 0.1 1"/>
-    </material>
-    <material name="blue">
-        <color rgba="0.2 0.2 1 1"/>
-    </material>
-    <material name="black">
-        <color rgba="0 0 0 1"/>
-    </material>
-    <!-- BASE LINK -->
-    <link name="base_link">
-    </link>
-    <!-- CHASSIS LINK -->
-    <joint name="chassis_joint" type="fixed">
-        <parent link="base_link"/>
-        <child link="chassis"/>
-        <origin xyz="-0.1 0 0"/>
-    </joint>
-    <link name="chassis">
-        <visual>
-            <origin xyz="0.15 0 0.075"/>
-            <geometry>
-                <box size="0.3 0.3 0.15"/>
-            </geometry>
-            <material name="white"/>
-        </visual>
-        <collision>
-            <origin xyz="0.15 0 0.075"/>
-            <geometry>
-                <box size="0.3 0.3 0.15"/>
-            </geometry>
-        </collision>
-        <xacro:inertial_box mass="0.5" x="0.3" y="0.3" z="0.15">
-            <origin xyz="0.15 0 0.075" rpy="0 0 0"/>
-        </xacro:inertial_box>
-    </link>
-    <gazebo reference="chassis">
-        <material>Gazebo/White</material>
-    </gazebo>
-    <!-- LEFT WHEEL LINK -->
-    <joint name="left_wheel_joint" type="continuous">
-        <parent link="base_link"/>
-        <child link="left_wheel"/>
-        <origin xyz="0 0.175 0" rpy="-${pi/2} 0 0" />
-        <axis xyz="0 0 1"/>
-    </joint>
-    <link name="left_wheel">
-        <visual>
-            <geometry>
-                <cylinder radius="0.05" length="0.04"/>
-            </geometry>
-            <material name="blue"/>
-        </visual>
-        <collision>
-            <geometry>
-                <cylinder radius="0.05" length="0.04"/>
-            </geometry>
-        </collision>
-        <xacro:inertial_cylinder mass="0.1" length="0.04" radius="0.05">
-            <origin xyz="0 0 0" rpy="0 0 0"/>
-        </xacro:inertial_cylinder>
-    </link>
-    <!-- RIGHT WHEEL LINK -->
-    <joint name="right_wheel_joint" type="continuous">
-        <parent link="base_link"/>
-        <child link="right_wheel"/>
-        <origin xyz="0 -0.175 0" rpy="${pi/2} 0 0" />
-        <axis xyz="0 0 -1"/>
-    </joint>
-    <link name="right_wheel">
-        <visual>
-            <geometry>
-                <cylinder radius="0.05" length="0.04"/>
-            </geometry>
-            <material name="blue"/>
-        </visual>
-        <collision>
-            <geometry>
-                <cylinder radius="0.05" length="0.04"/>
-            </geometry>
-        </collision>
-        <xacro:inertial_cylinder mass="0.1" length="0.04" radius="0.05">
-            <origin xyz="0 0 0" rpy="0 0 0"/>
-        </xacro:inertial_cylinder>
-    </link>
-    <!-- CASTER WHEEL LINK -->
-    <joint name="caster_wheel_joint" type="fixed">
-        <parent link="chassis"/>
-        <child link="caster_wheel"/>
-        <origin xyz="0.24 0 0"/>
-    </joint>
-    <link name="caster_wheel">
-        <visual>
-            <geometry>
-                <sphere radius="0.05"/>
-            </geometry>
-            <material name="black"/>
-        </visual>
-        <collision>
-            <geometry>
-                <sphere radius="0.05"/>
-            </geometry>
-        </collision>
-        <xacro:inertial_sphere mass="0.1" radius="0.05">
-            <origin xyz="0 0 0" rpy="0 0 0"/>
-        </xacro:inertial_sphere>
-    </link>
-    <gazebo reference="caster_wheel">
-        <material>Gazebo/Black</material>
-        <mu1 value="0.001"/>
-        <mu2 value="0.001"/>
-    </gazebo>
+    <xacro:macro name="robot_core" params="">
+        <material name="white">
+            <color rgba="1 1 1 1" />
+        </material>
+        <material name="orange">
+            <color rgba="1 0.3 0.1 1"/>
+        </material>
+        <material name="blue">
+            <color rgba="0.2 0.2 1 1"/>
+        </material>
+        <material name="black">
+            <color rgba="0 0 0 1"/>
+        </material>
+        <!-- BASE LINK -->
+        <link name="base_link">
+        </link>
+        <!-- CHASSIS LINK -->
+        <joint name="chassis_joint" type="fixed">
+            <parent link="base_link"/>
+            <child link="chassis"/>
+            <origin xyz="-0.1 0 0"/>
+        </joint>
+        <link name="chassis">
+            <visual>
+                <origin xyz="0.15 0 0.075"/>
+                <geometry>
+                    <box size="0.3 0.3 0.15"/>
+                </geometry>
+                <material name="white"/>
+            </visual>
+            <collision>
+                <origin xyz="0.15 0 0.075"/>
+                <geometry>
+                    <box size="0.3 0.3 0.15"/>
+                </geometry>
+            </collision>
+            <xacro:inertial_box mass="0.5" x="0.3" y="0.3" z="0.15">
+                <origin xyz="0.15 0 0.075" rpy="0 0 0"/>
+            </xacro:inertial_box>
+        </link>
+        <gazebo reference="chassis">
+            <material>Gazebo/White</material>
+        </gazebo>
+        <!-- LEFT WHEEL LINK -->
+        <joint name="left_wheel_joint" type="continuous">
+            <parent link="base_link"/>
+            <child link="left_wheel"/>
+            <origin xyz="0 0.175 0" rpy="-${pi/2} 0 0" />
+            <axis xyz="0 0 1"/>
+        </joint>
+        <link name="left_wheel">
+            <visual>
+                <geometry>
+                    <cylinder radius="0.05" length="0.04"/>
+                </geometry>
+                <material name="blue"/>
+            </visual>
+            <collision>
+                <geometry>
+                    <cylinder radius="0.05" length="0.04"/>
+                </geometry>
+            </collision>
+            <xacro:inertial_cylinder mass="0.1" length="0.04" radius="0.05">
+                <origin xyz="0 0 0" rpy="0 0 0"/>
+            </xacro:inertial_cylinder>
+        </link>
+        <!-- RIGHT WHEEL LINK -->
+        <joint name="right_wheel_joint" type="continuous">
+            <parent link="base_link"/>
+            <child link="right_wheel"/>
+            <origin xyz="0 -0.175 0" rpy="${pi/2} 0 0" />
+            <axis xyz="0 0 -1"/>
+        </joint>
+        <link name="right_wheel">
+            <visual>
+                <geometry>
+                    <cylinder radius="0.05" length="0.04"/>
+                </geometry>
+                <material name="blue"/>
+            </visual>
+            <collision>
+                <geometry>
+                    <cylinder radius="0.05" length="0.04"/>
+                </geometry>
+            </collision>
+            <xacro:inertial_cylinder mass="0.1" length="0.04" radius="0.05">
+                <origin xyz="0 0 0" rpy="0 0 0"/>
+            </xacro:inertial_cylinder>
+        </link>
+        <!-- CASTER WHEEL LINK -->
+        <joint name="caster_wheel_joint" type="fixed">
+            <parent link="chassis"/>
+            <child link="caster_wheel"/>
+            <origin xyz="0.24 0 0"/>
+        </joint>
+        <link name="caster_wheel">
+            <visual>
+                <geometry>
+                    <sphere radius="0.05"/>
+                </geometry>
+                <material name="black"/>
+            </visual>
+            <collision>
+                <geometry>
+                    <sphere radius="0.05"/>
+                </geometry>
+            </collision>
+            <xacro:inertial_sphere mass="0.1" radius="0.05">
+                <origin xyz="0 0 0" rpy="0 0 0"/>
+            </xacro:inertial_sphere>
+        </link>
+        <gazebo reference="caster_wheel">
+            <material>Gazebo/Black</material>
+            <mu1 value="0.001"/>
+            <mu2 value="0.001"/>
+        </gazebo>
+    </xacro:macro>
 </robot>
